Commit message: "Update the LQR controller."

File: install/balance_bot/share/balance_bot/urdf/bot_with_sensors.xacro (robot description, xacro)
@@ -1,59 +1 @@
-<?xml version="1.0"?>
-<robot name="wheel_leg_robot" xmlns:xacro="http://www.ros.org/wiki/xacro">
-  <!-- 包含基础模型 -->
-  <xacro:include filename="$(find balance_bot)/urdf/wheel_leg_initial_pose.xacro" />
-  <!-- 添加IMU传感器插件 -->
-  <gazebo reference="base_link">
-    <sensor name="imu_sensor" type="imu">
-      <always_on>true</always_on>
-      <update_rate>100</update_rate>
-      <imu>
-        <noise>
-          <type>gaussian</type>
-          <rate>
-            <mean>0.0</mean>
-            <stddev>0.0002</stddev>
-            <bias_mean>0.0000075</bias_mean>
-            <bias_stddev>0.0000008</bias_stddev>
-          </rate>
-          <accel>
-            <mean>0.0</mean>
-            <stddev>0.017</stddev>
-            <bias_mean>0.1</bias_mean>
-            <bias_stddev>0.001</bias_stddev>
-          </accel>
-        </noise>
-      </imu>
-    </sensor>
-  </gazebo>
-  <!-- IMU ROS插件 -->
-  <gazebo>
-    <plugin filename="libgazebo_ros_imu_sensor.so" name="imu_plugin">
-      <topicName>/imu</topicName>
-      <bodyName>base_link</bodyName>
-      <updateRateHZ>100.0</updateRateHZ>
-      <gravityZ>9.81</gravityZ>
-      <xyzOffset>0 0 0</xyzOffset>
-      <rpyOffset>0 0 0</rpyOffset>
-      <frameName>base_link</frameName>
-    </plugin>
-  </gazebo>
-  <!-- 里程计插件 -->
-  <gazebo>
-    <plugin filename="libgazebo_ros_diff_drive.so" name="diff_drive_controller">
-      <ros>
-        <namespace>/wheel_leg_robot</namespace>
-      </ros>
-      <update_rate>50</update_rate>
-      <left_joint>left_wheel_joint</left_joint>
-      <right_joint>right_wheel_joint</right_joint>
-      <wheel_separation>0.3</wheel_separation>
-      <wheel_diameter>0.16</wheel_diameter>
-      <max_wheel_torque>20</max_wheel_torque>
-      <command_topic>/cmd_vel</command_topic>
-      <odometry_topic>odom</odometry_topic>
-      <odometry_frame>odom</odometry_frame>
-      <robot_base_frame>base_link</robot_base_frame>
-    </plugin>
-  </gazebo>
-</robot>
+/home/nuaawzh/dev_ws/src/balance_bot/urdf/bot_with_sensors.xacro

File: install/balance_bot/share/balance_bot/urdf/leg_initial_pose_module.xacro (robot description, xacro)
@@ -1,161 +1 @@
-<?xml version="1.0"?>
-<robot xmlns:xacro="http://www.ros.org/wiki/xacro">
-  <xacro:macro name="leg_initial_pose_module" params="prefix parent x y z mirror">
-    <!-- 定义几何参数 -->
-    <xacro:property name="thigh_length" value="0.35" />    <!-- 大腿长度 -->
-    <xacro:property name="shank_length" value="0.3" />     <!-- 小腿长度 -->
-    <xacro:property name="leg_diameter" value="0.02" />
-    <xacro:property name="wheel_radius" value="0.08" />
-    <xacro:property name="wheel_thickness" value="0.04" />
-    <!-- 初始角度参数 -->
-    <xacro:property name="initial_hip_angle" value="${-pi/3}" />  <!-- 大腿与地面法线成60度角（-60度） -->
-    <xacro:property name="initial_knee_angle" value="${2*pi/3}" /> <!-- 膝关节角度，使轮子投影与髋关节重合 -->
-    <!-- 镜像因子 -->
-    <xacro:property name="mirror_factor" value="${-1 if mirror else 1}" />
-    <!-- ========== 大腿 (Thigh) ========== -->
-    <link name="${prefix}_thigh">
-      <visual>
-        <geometry>
-          <cylinder radius="${leg_diameter/2}" length="${thigh_length}"/>
-        </geometry>
-        <material name="red">
-          <color rgba="0.8 0 0 1"/>
-        </material>
-        <origin xyz="0 0 ${-thigh_length/2}" rpy="0 0 0"/>
-      </visual>
-      <collision>
-        <geometry>
-          <cylinder radius="${leg_diameter/2}" length="${thigh_length}"/>
-        </geometry>
-        <origin xyz="0 0 ${-thigh_length/2}" rpy="0 0 0"/>
-      </collision>
-      <inertial>
-        <mass value="0.4"/>
-        <inertia ixx="0.003" ixy="0.0" ixz="0.0" iyy="0.003" iyz="0.0" izz="0.0002"/>
-      </inertial>
-    </link>
-    <!-- 大腿与机体的关节 (髋关节电机) - 初始角度为-60度 -->
-    <joint name="${prefix}_hip_joint" type="revolute">
-      <parent link="${parent}"/>
-      <child link="${prefix}_thigh"/>
-      <origin xyz="${x} ${y} ${z}" rpy="0 0 0"/>
-      <axis xyz="0 1 0"/>
-      <limit lower="-2.0" upper="1.0" effort="30.0" velocity="3.0"/>
-      <!-- 设置初始位置 -->
-      <xacro:if value="${mirror}">
-        <origin rpy="0 ${initial_hip_angle} 0" xyz="${x} ${y} ${z}"/>
-      </xacro:if>
-      <xacro:unless value="${mirror}">
-        <origin rpy="0 ${initial_hip_angle} 0" xyz="${x} ${y} ${z}"/>
-      </xacro:unless>
-    </joint>
-    <!-- ========== 小腿 (Shank) ========== -->
-    <link name="${prefix}_shank">
-      <visual>
-        <geometry>
-          <cylinder radius="${leg_diameter/2}" length="${shank_length}"/>
-        </geometry>
-        <material name="green">
-          <color rgba="0 0.8 0 1"/>
-        </material>
-        <origin xyz="0 0 ${-shank_length/2}" rpy="0 0 0"/>
-      </visual>
-      <collision>
-        <geometry>
-          <cylinder radius="${leg_diameter/2}" length="${shank_length}"/>
-        </geometry>
-        <origin xyz="0 0 ${-shank_length/2}" rpy="0 0 0"/>
-      </collision>
-      <inertial>
-        <mass value="0.3"/>
-        <inertia ixx="0.002" ixy="0.0" ixz="0.0" iyy="0.002" iyz="0.0" izz="0.0001"/>
-      </inertial>
-    </link>
-    <!-- 小腿与大腿的关节 (膝关节电机) - 初始角度为120度 -->
-    <joint name="${prefix}_knee_joint" type="revolute">
-      <parent link="${prefix}_thigh"/>
-      <child link="${prefix}_shank"/>
-      <origin xyz="0 0 ${-thigh_length}" rpy="0 0 0"/>
-      <axis xyz="0 1 0"/>
-      <limit lower="0.5" upper="2.5" effort="25.0" velocity="3.0"/>
-      <!-- 设置初始位置 -->
-      <xacro:if value="${mirror}">
-        <origin rpy="0 ${initial_knee_angle} 0" xyz="0 0 ${-thigh_length}"/>
-      </xacro:if>
-      <xacro:unless value="${mirror}">
-        <origin rpy="0 ${initial_knee_angle} 0" xyz="0 0 ${-thigh_length}"/>
-      </xacro:unless>
-    </joint>
-    <!-- ========== 轮子 (Wheel) ========== -->
-    <link name="${prefix}_wheel">
-      <visual>
-        <geometry>
-          <cylinder radius="${wheel_radius}" length="${wheel_thickness}"/>
-        </geometry>
-        <material name="black">
-          <color rgba="0 0 0 1"/>
-        </material>
-      </visual>
-      <collision>
-        <geometry>
-          <cylinder radius="${wheel_radius}" length="${wheel_thickness}"/>
-        </geometry>
-      </collision>
-      <inertial>
-        <mass value="0.5"/>
-        <inertia ixx="0.002" ixy="0.0" ixz="0.0" iyy="0.001" iyz="0.0" izz="0.002"/>
-      </inertial>
-    </link>
-    <!-- 轮子与小腿的关节 (无刷电机) -->
-    <joint name="${prefix}_wheel_joint" type="continuous">
-      <parent link="${prefix}_shank"/>
-      <child link="${prefix}_wheel"/>
-      <origin xyz="0 0 ${-shank_length}" rpy="${pi/2} 0 0"/>
-      <axis xyz="0 1 0"/>
-    </joint>
-    <!-- ========== 传输定义 ========== -->
-    <!-- 髋关节传输 -->
-    <transmission name="${prefix}_hip_trans">
-      <type>transmission_interface/SimpleTransmission</type>
-      <joint name="${prefix}_hip_joint">
-        <hardwareInterface>PositionJointInterface</hardwareInterface>
-      </joint>
-      <actuator name="${prefix}_hip_motor">
-        <hardwareInterface>PositionJointInterface</hardwareInterface>
-        <mechanicalReduction>1</mechanicalReduction>
-      </actuator>
-    </transmission>
-    <!-- 膝关节传输 -->
-    <transmission name="${prefix}_knee_trans">
-      <type>transmission_interface/SimpleTransmission</type>
-      <joint name="${prefix}_knee_joint">
-        <hardwareInterface>PositionJointInterface</hardwareInterface>
-      </joint>
-      <actuator name="${prefix}_knee_motor">
-        <hardwareInterface>PositionJointInterface</hardwareInterface>
-        <mechanicalReduction>1</mechanicalReduction>
-      </actuator>
-    </transmission>
-    <!-- 轮子关节传输 -->
-    <transmission name="${prefix}_wheel_trans">
-      <type>transmission_interface/SimpleTransmission</type>
-      <joint name="${prefix}_wheel_joint">
-        <hardwareInterface>VelocityJointInterface</hardwareInterface>
-      </joint>
-      <actuator name="${prefix}_wheel_motor">
-        <hardwareInterface>VelocityJointInterface</hardwareInterface>
-        <mechanicalReduction>1</mechanicalReduction>
-      </actuator>
-    </transmission>
-    <!-- Gazebo材质 -->
-    <gazebo reference="${prefix}_thigh">
-      <material>Gazebo/Red</material>
-    </gazebo>
-    <gazebo reference="${prefix}_shank">
-      <material>Gazebo/Green</material>
-    </gazebo>
-    <gazebo reference="${prefix}_wheel">
-      <material>Gazebo/Black</material>
-    </gazebo>
-  </xacro:macro>
-</robot>
+/home/nuaawzh/dev_ws/src/balance_bot/urdf/leg_initial_pose_module.xacro

File: install/balance_bot/share/balance_bot/urdf/wheel_leg_initial_pose.xacro (robot description, xacro)
@@ -1,55 +1 @@
-<?xml version="1.0"?>
-<robot name="wheel_leg_initial_pose" xmlns:xacro="http://www.ros.org/wiki/xacro">
-  <!-- 包含宏定义 -->
-  <xacro:include filename="$(find balance_bot)/urdf/leg_initial_pose_module.xacro" />
-  <!-- 定义机器人参数 -->
-  <xacro:property name="body_length" value="0.4" />
-  <xacro:property name="body_width" value="0.3" />
-  <xacro:property name="body_height" value="0.15" />
-  <!-- 机器人主体 -->
-  <link name="base_link">
-    <visual>
-      <geometry>
-        <box size="${body_length} ${body_width} ${body_height}"/>
-      </geometry>
-      <material name="blue">
-        <color rgba="0 0 0.8 1"/>
-      </material>
-    </visual>
-    <collision>
-      <geometry>
-        <box size="${body_length} ${body_width} ${body_height}"/>
-      </geometry>
-    </collision>
-    <inertial>
-      <mass value="2.0"/>
-      <inertia ixx="0.02" ixy="0.0" ixz="0.0" iyy="0.02" iyz="0.0" izz="0.02"/>
-    </inertial>
-  </link>
-  <!-- 添加左侧腿 -->
-  <xacro:leg_initial_pose_module
-    prefix="left"
-    parent="base_link"
-    x="${0}"
-    y="${body_width/2}"
-    z="0"
-    mirror="false" />
-  <!-- 添加右侧腿 -->
-  <xacro:leg_initial_pose_module
-    prefix="right"
-    parent="base_link"
-    x="${0}"
-    y="${-body_width/2}"
-    z="0"
-    mirror="true" />
-  <!-- Gazebo插件 -->
-  <gazebo reference="base_link">
-    <material>Gazebo/Blue</material>
-  </gazebo>
-  <!-- Gazebo ROS控制插件 -->
-  <gazebo>
-    <plugin name="gazebo_ros_control" filename="libgazebo_ros_control.so">
-      <robotNamespace>/wheel_leg_initial_pose</robotNamespace>
-    </plugin>
-  </gazebo>
-</robot>
+/home/nuaawzh/dev_ws/src/balance_bot/urdf/wheel_leg_initial_pose.xacro
