Commit message: "Update the LQR controller."

File: src/balance_bot/urdf/bot_with_sensors.xacro (robot description, xacro)
@@ -8,38 +8,65 @@
       <always_on>true</always_on>
       <update_rate>100</update_rate>
+      <topic>imu</topic>
       <imu>
-        <noise>
-          <type>gaussian</type>
-          <rate>
-            <mean>0.0</mean>
-            <stddev>0.0002</stddev>
-            <bias_mean>0.0000075</bias_mean>
-            <bias_stddev>0.0000008</bias_stddev>
-          </rate>
-          <accel>
-            <mean>0.0</mean>
-            <stddev>0.017</stddev>
-            <bias_mean>0.1</bias_mean>
-            <bias_stddev>0.001</bias_stddev>
-          </accel>
-        </noise>
+        <angular_velocity>
+          <x>
+            <noise type="gaussian">
+              <mean>0.0</mean>
+              <stddev>0.0002</stddev>
+              <bias_mean>0.0000075</bias_mean>
+              <bias_stddev>0.0000008</bias_stddev>
+            </noise>
+          </x>
+          <y>
+            <noise type="gaussian">
+              <mean>0.0</mean>
+              <stddev>0.0002</stddev>
+              <bias_mean>0.0000075</bias_mean>
+              <bias_stddev>0.0000008</bias_stddev>
+            </noise>
+          </y>
+          <z>
+            <noise type="gaussian">
+              <mean>0.0</mean>
+              <stddev>0.0002</stddev>
+              <bias_mean>0.0000075</bias_mean>
+              <bias_stddev>0.0000008</bias_stddev>
+            </noise>
+          </z>
+        </angular_velocity>
+        <linear_acceleration>
+          <x>
+            <noise type="gaussian">
+              <mean>0.0</mean>
+              <stddev>0.017</stddev>
+              <bias_mean>0.1</bias_mean>
+              <bias_stddev>0.001</bias_stddev>
+            </noise>
+          </x>
+          <y>
+            <noise type="gaussian">
+              <mean>0.0</mean>
+              <stddev>0.017</stddev>
+              <bias_mean>0.1</bias_mean>
+              <bias_stddev>0.001</bias_stddev>
+            </noise>
+          </y>
+          <z>
+            <noise type="gaussian">
+              <mean>0.0</mean>
+              <stddev>0.017</stddev>
+              <bias_mean>0.1</bias_mean>
+              <bias_stddev>0.001</bias_stddev>
+            </noise>
+          </z>
+        </linear_acceleration>
       </imu>
     </sensor>
   </gazebo>
-  <!-- IMU ROS插件 -->
+  <!-- Legacy IMU plugin removed -->
+  <!-- 里程计插件 (已注释，避免与 customized force control 冲突)
   <gazebo>
-    <plugin filename="libgz_sim_imu_system.so" name="imu_plugin">
-      <topicName>/imu</topicName>
-      <bodyName>base_link</bodyName>
-      <updateRateHZ>100.0</updateRateHZ>
-      <gravityZ>9.81</gravityZ>
-      <xyzOffset>0 0 0</xyzOffset>
-      <rpyOffset>0 0 0</rpyOffset>
-      <frameName>base_link</frameName>
-    </plugin>
-  </gazebo>
-  <!-- 里程计插件 -->
-  <gazebo>
-    <plugin filename="libgz_sim_diff_drive_system.so" name="diff_drive_controller">
+    <plugin filename="libgz_sim_diff_drive_system.so" name="gz::sim::systems::DiffDrive">
       <ros>
         <namespace>/wheel_leg_robot</namespace>
@@ -57,3 +84,4 @@
     </plugin>
   </gazebo>
+  -->
 </robot>

File: src/balance_bot/urdf/leg_initial_pose_module.xacro (robot description, xacro)
@@ -99,4 +99,5 @@
           <color rgba="0 0 0 1"/>
         </material>
+        <origin xyz="0 0 0" rpy="${pi/2} 0 0"/>
       </visual>
       <collision>
@@ -104,8 +105,10 @@
           <cylinder radius="${wheel_radius}" length="${wheel_thickness}"/>
         </geometry>
+        <origin xyz="0 0 0" rpy="${pi/2} 0 0"/>
       </collision>
       <inertial>
         <mass value="0.982"/>
-        <inertia ixx="0.002" ixy="0.0" ixz="0.0" iyy="0.002" iyz="0.0" izz="0.001"/> <!-- izz对应旋转轴惯量 -->
+        <!-- Adjusted inertia for Y-axis rotation: iyy is now the axis of rotation -->
+        <inertia ixx="0.002" ixy="0.0" ixz="0.0" iyy="0.001" iyz="0.0" izz="0.002"/>
       </inertial>
     </link>
@@ -114,5 +117,5 @@
       <parent link="${prefix}_shank"/>
       <child link="${prefix}_wheel"/>
-      <origin xyz="0 0 ${-shank_length}" rpy="${pi/2} 0 0"/>
+      <origin xyz="0 0 ${-shank_length}" rpy="0 0 0"/>
       <axis xyz="0 1 0"/>
     </joint>

File: src/balance_bot/urdf/wheel_leg_initial_pose.xacro (robot description, xacro)
@@ -52,4 +52,65 @@
     z="0"
     mirror="true" />
+  <ros2_control name="GazeboSystem" type="system">
+    <hardware>
+      <plugin>gz_ros2_control/GazeboSimSystem</plugin>
+    </hardware>
+    <!-- Left Leg -->
+    <joint name="left_hip_joint">
+      <command_interface name="effort">
+        <param name="min">-30</param>
+        <param name="max">30</param>
+      </command_interface>
+      <state_interface name="position"/>
+      <state_interface name="velocity"/>
+      <state_interface name="effort"/>
+    </joint>
+    <joint name="left_knee_joint">
+      <command_interface name="effort">
+        <param name="min">-25</param>
+        <param name="max">25</param>
+      </command_interface>
+      <state_interface name="position"/>
+      <state_interface name="velocity"/>
+      <state_interface name="effort"/>
+    </joint>
+    <joint name="left_wheel_joint">
+      <command_interface name="effort">
+        <param name="min">-15</param>
+        <param name="max">15</param>
+      </command_interface>
+      <state_interface name="position"/>
+      <state_interface name="velocity"/>
+      <state_interface name="effort"/>
+    </joint>
+    <!-- Right Leg -->
+    <joint name="right_hip_joint">
+      <command_interface name="effort">
+        <param name="min">-30</param>
+        <param name="max">30</param>
+      </command_interface>
+      <state_interface name="position"/>
+      <state_interface name="velocity"/>
+      <state_interface name="effort"/>
+    </joint>
+    <joint name="right_knee_joint">
+      <command_interface name="effort">
+        <param name="min">-25</param>
+        <param name="max">25</param>
+      </command_interface>
+      <state_interface name="position"/>
+      <state_interface name="velocity"/>
+      <state_interface name="effort"/>
+    </joint>
+    <joint name="right_wheel_joint">
+      <command_interface name="effort">
+        <param name="min">-15</param>
+        <param name="max">15</param>
+      </command_interface>
+      <state_interface name="position"/>
+      <state_interface name="velocity"/>
+      <state_interface name="effort"/>
+    </joint>
+  </ros2_control>
   <!-- Gazebo插件 -->
   <gazebo reference="base_link">
@@ -58,6 +119,6 @@
   <!-- Gazebo ROS控制插件 -->
   <gazebo>
-    <plugin name="gazebo_ros_control" filename="libgz_ros2_control-system.so">
-      <robotNamespace>/wheel_leg_initial_pose</robotNamespace>
+    <plugin name="gz_ros2_control::GazeboSimROS2ControlPlugin" filename="libgz_ros2_control-system.so">
+      <parameters>$(find balance_bot)/config/controllers.yaml</parameters>
     </plugin>
   </gazebo>

Commit message: "Update the LQR controller."

File: src/balance_bot/urdf/bot_with_sensors.xacro (robot description, xacro)
@@ -7,7 +7,18 @@
     <sensor name="imu_sensor" type="imu">
       <always_on>true</always_on>
-      <update_rate>100</update_rate>
-      <topic>imu</topic>
-      <imu>
+      <update_rate>1000</update_rate>
+      <!-- Gazebo内部发布IMU数据的话题，桥接会连接到这里 -->
+      <topic>/imu</topic>
+      <plugin filename="libgz-sim-imu-system.so" name="gz::sim::systems::Imu">
+        <!-- 注意：这里的是插件内部参数，与你上面的<imu>标签是两套东西。
+             下面的噪声配置是为插件准备的，格式也不同。-->
+        <topic>/imu</topic>
+        <noise type="gaussian">
+          <mean>0.0</mean>
+          <stddev>0.0002</stddev>
+        </noise>
+        <!-- 为了快速验证，你可以先注释掉下面详细的噪声配置，
+             等传感器能工作后再来细化。 -->
+        <!--
         <angular_velocity>
           <x>
@@ -15,6 +26,4 @@
               <mean>0.0</mean>
               <stddev>0.0002</stddev>
-              <bias_mean>0.0000075</bias_mean>
-              <bias_stddev>0.0000008</bias_stddev>
             </noise>
           </x>
@@ -23,6 +32,4 @@
               <mean>0.0</mean>
               <stddev>0.0002</stddev>
-              <bias_mean>0.0000075</bias_mean>
-              <bias_stddev>0.0000008</bias_stddev>
             </noise>
           </y>
@@ -31,6 +38,4 @@
               <mean>0.0</mean>
               <stddev>0.0002</stddev>
-              <bias_mean>0.0000075</bias_mean>
-              <bias_stddev>0.0000008</bias_stddev>
             </noise>
           </z>
@@ -41,6 +46,4 @@
               <mean>0.0</mean>
               <stddev>0.017</stddev>
-              <bias_mean>0.1</bias_mean>
-              <bias_stddev>0.001</bias_stddev>
             </noise>
           </x>
@@ -49,6 +52,4 @@
               <mean>0.0</mean>
               <stddev>0.017</stddev>
-              <bias_mean>0.1</bias_mean>
-              <bias_stddev>0.001</bias_stddev>
             </noise>
           </y>
@@ -57,10 +58,9 @@
               <mean>0.0</mean>
               <stddev>0.017</stddev>
-              <bias_mean>0.1</bias_mean>
-              <bias_stddev>0.001</bias_stddev>
             </noise>
           </z>
         </linear_acceleration>
-      </imu>
+        -->
+      </plugin>
     </sensor>
   </gazebo>

File: src/balance_bot/urdf/leg_initial_pose_module.xacro (robot description, xacro)
@@ -43,5 +43,5 @@
       <origin xyz="${x} ${y} ${z}" rpy="0 0 0"/>
       <axis xyz="0 1 0"/>
-      <limit lower="-3.0" upper="1.0" effort="30.0" velocity="3.0"/>
+      <limit lower="-3.0" upper="1.0" effort="30.0" velocity="10.0"/>
       <!-- 设置初始位置 -->
       <xacro:if value="${mirror}">
@@ -81,5 +81,5 @@
       <origin xyz="0 0 ${-thigh_length}" rpy="0 0 0"/>
       <axis xyz="0 1 0"/>
-      <limit lower="0.0" upper="3.0" effort="25.0" velocity="3.0"/>
+      <limit lower="0.0" upper="3.0" effort="25.0" velocity="10.0"/>
       <!-- 设置初始位置 -->
       <xacro:if value="${mirror}">
@@ -109,9 +109,9 @@
       <inertial>
         <mass value="0.982"/>
-        <!-- Adjusted inertia for Y-axis rotation: iyy is now the axis of rotation -->
         <inertia ixx="0.002" ixy="0.0" ixz="0.0" iyy="0.001" iyz="0.0" izz="0.002"/>
       </inertial>
     </link>
     <!-- 轮子与腿的关节 (无刷电机) -->
+    <!-- 修正轮子轴向，假设原方向错误 -->
     <joint name="${prefix}_wheel_joint" type="continuous">
       <parent link="${prefix}_shank"/>
