Commit message: "Update the LQR controller."

File: src/balance_bot/urdf/leg_initial_pose_module.xacro (robot description, xacro)
@@ -3,12 +3,13 @@
   <xacro:macro name="leg_initial_pose_module" params="prefix parent x y z mirror">
     <!-- 定义几何参数 -->
-    <xacro:property name="thigh_length" value="0.35" />    <!-- 大腿长度 -->
-    <xacro:property name="shank_length" value="0.3" />     <!-- 小腿长度 -->
-    <xacro:property name="leg_diameter" value="0.02" />
-    <xacro:property name="wheel_radius" value="0.08" />
+    <xacro:property name="thigh_length" value="0.23" />    <!-- 大腿长度 230mm -->
+    <xacro:property name="shank_length" value="0.287" />   <!-- 小腿长度 287mm -->
+    <xacro:property name="leg_diameter" value="0.04" />
+    <xacro:property name="wheel_radius" value="0.058" />
     <xacro:property name="wheel_thickness" value="0.04" />
     <!-- 初始角度参数 -->
-    <xacro:property name="initial_hip_angle" value="${-pi/3}" />  <!-- 大腿与地面法线成60度角（-60度） -->
-    <xacro:property name="initial_knee_angle" value="${2*pi/3}" /> <!-- 膝关节角度，使轮子投影与髋关节重合 -->
+    <!-- 髋关节高度 0.176 => Hip: -1.55 rad, Knee: 2.48 rad -->
+    <xacro:property name="initial_hip_angle" value="-1.55" />
+    <xacro:property name="initial_knee_angle" value="2.48" />
     <!-- 镜像因子 -->
     <xacro:property name="mirror_factor" value="${-1 if mirror else 1}" />
@@ -31,9 +32,10 @@
       </collision>
       <inertial>
-        <mass value="0.4"/>
-        <inertia ixx="0.003" ixy="0.0" ixz="0.0" iyy="0.003" iyz="0.0" izz="0.0002"/>
+        <mass value="1.02"/> <!-- 总腿重2.047，平均分配 -->
+        <inertia ixx="0.009" ixy="0.0" ixz="0.0" iyy="0.009" iyz="0.0" izz="0.001"/>
+        <origin xyz="0 0 ${-thigh_length/2}" rpy="0 0 0"/>
       </inertial>
     </link>
-    <!-- 大腿与机体的关节 (髋关节电机) - 初始角度为-60度 -->
+    <!-- 大腿与机体的关节 (髋关节电机) -->
     <joint name="${prefix}_hip_joint" type="revolute">
       <parent link="${parent}"/>
@@ -41,5 +43,5 @@
       <origin xyz="${x} ${y} ${z}" rpy="0 0 0"/>
       <axis xyz="0 1 0"/>
-      <limit lower="-2.0" upper="1.0" effort="30.0" velocity="3.0"/>
+      <limit lower="-3.0" upper="1.0" effort="30.0" velocity="3.0"/>
       <!-- 设置初始位置 -->
       <xacro:if value="${mirror}">
@@ -68,9 +70,10 @@
       </collision>
       <inertial>
-        <mass value="0.3"/>
-        <inertia ixx="0.002" ixy="0.0" ixz="0.0" iyy="0.002" iyz="0.0" izz="0.0001"/>
+        <mass value="1.027"/> <!-- 补足到总重2.047 -->
+        <inertia ixx="0.009" ixy="0.0" ixz="0.0" iyy="0.009" iyz="0.0" izz="0.001"/>
+        <origin xyz="0 0 ${-shank_length/2}" rpy="0 0 0"/>
       </inertial>
     </link>
-    <!-- 小腿与大腿的关节 (膝关节电机) - 初始角度为120度 -->
+    <!-- 小腿与大腿的关节 (膝关节电机) -->
     <joint name="${prefix}_knee_joint" type="revolute">
       <parent link="${prefix}_thigh"/>
@@ -78,5 +81,5 @@
       <origin xyz="0 0 ${-thigh_length}" rpy="0 0 0"/>
       <axis xyz="0 1 0"/>
-      <limit lower="0.5" upper="2.5" effort="25.0" velocity="3.0"/>
+      <limit lower="0.0" upper="3.0" effort="25.0" velocity="3.0"/>
       <!-- 设置初始位置 -->
       <xacro:if value="${mirror}">
@@ -103,9 +106,9 @@
       </collision>
       <inertial>
-        <mass value="0.5"/>
-        <inertia ixx="0.002" ixy="0.0" ixz="0.0" iyy="0.001" iyz="0.0" izz="0.002"/>
+        <mass value="0.982"/>
+        <inertia ixx="0.002" ixy="0.0" ixz="0.0" iyy="0.002" iyz="0.0" izz="0.001"/> <!-- izz对应旋转轴惯量 -->
       </inertial>
     </link>
-    <!-- 轮子与小腿的关节 (无刷电机) -->
+    <!-- 轮子与腿的关节 (无刷电机) -->
     <joint name="${prefix}_wheel_joint" type="continuous">
       <parent link="${prefix}_shank"/>
@@ -119,8 +122,8 @@
       <type>transmission_interface/SimpleTransmission</type>
       <joint name="${prefix}_hip_joint">
-        <hardwareInterface>PositionJointInterface</hardwareInterface>
+        <hardwareInterface>EffortJointInterface</hardwareInterface>
       </joint>
       <actuator name="${prefix}_hip_motor">
-        <hardwareInterface>PositionJointInterface</hardwareInterface>
+        <hardwareInterface>EffortJointInterface</hardwareInterface>
         <mechanicalReduction>1</mechanicalReduction>
       </actuator>
@@ -130,8 +133,8 @@
       <type>transmission_interface/SimpleTransmission</type>
       <joint name="${prefix}_knee_joint">
-        <hardwareInterface>PositionJointInterface</hardwareInterface>
+        <hardwareInterface>EffortJointInterface</hardwareInterface>
       </joint>
       <actuator name="${prefix}_knee_motor">
-        <hardwareInterface>PositionJointInterface</hardwareInterface>
+        <hardwareInterface>EffortJointInterface</hardwareInterface>
         <mechanicalReduction>1</mechanicalReduction>
       </actuator>
@@ -141,8 +144,8 @@
       <type>transmission_interface/SimpleTransmission</type>
       <joint name="${prefix}_wheel_joint">
-        <hardwareInterface>VelocityJointInterface</hardwareInterface>
+        <hardwareInterface>EffortJointInterface</hardwareInterface>
       </joint>
       <actuator name="${prefix}_wheel_motor">
-        <hardwareInterface>VelocityJointInterface</hardwareInterface>
+        <hardwareInterface>EffortJointInterface</hardwareInterface>
         <mechanicalReduction>1</mechanicalReduction>
       </actuator>

File: src/balance_bot/urdf/wheel_leg_initial_pose.xacro (robot description, xacro)
@@ -5,5 +5,5 @@
   <!-- 定义机器人参数 -->
   <xacro:property name="body_length" value="0.4" />
-  <xacro:property name="body_width" value="0.3" />
+  <xacro:property name="body_width" value="0.35" /> <!-- Width 0.35 implies half-width 0.175 -->
   <xacro:property name="body_height" value="0.15" />
   <!-- 机器人主体 -->
@@ -23,6 +23,9 @@
     </collision>
     <inertial>
-      <mass value="2.0"/>
-      <inertia ixx="0.02" ixy="0.0" ixz="0.0" iyy="0.02" iyz="0.0" izz="0.02"/>
+      <mass value="15.0"/>
+      <!-- Pitch (y-axis) = 0.1125, Yaw (z-axis) = 0.05. Estimating Roll (x-axis) ~ 0.1 -->
+      <inertia ixx="0.1" ixy="0.0" ixz="0.0" iyy="0.1125" iyz="0.0" izz="0.05"/>
+      <!-- COM distance from hip axis is 0.05 -->
+      <origin xyz="0 0 0.05" rpy="0 0 0"/>
     </inertial>
   </link>

Commit message: "Update the LQR controller."

File: src/balance_bot/urdf/leg_initial_pose_module.xacro (robot description, xacro)
@@ -79,14 +79,7 @@
       <parent link="${prefix}_thigh"/>
       <child link="${prefix}_shank"/>
-      <origin xyz="0 0 ${-thigh_length}" rpy="0 0 0"/>
+      <origin rpy="0 ${initial_knee_angle} 0" xyz="0 0 ${-thigh_length}"/>
       <axis xyz="0 1 0"/>
       <limit lower="0.0" upper="3.0" effort="25.0" velocity="10.0"/>
-      <!-- 设置初始位置 -->
-      <xacro:if value="${mirror}">
-        <origin rpy="0 ${initial_knee_angle} 0" xyz="0 0 ${-thigh_length}"/>
-      </xacro:if>
-      <xacro:unless value="${mirror}">
-        <origin rpy="0 ${initial_knee_angle} 0" xyz="0 0 ${-thigh_length}"/>
-      </xacro:unless>
     </joint>
     <!-- ========== 轮子 (Wheel) ========== -->

Commit message: "Update the LQR controller, and failed."

File: src/balance_bot/urdf/leg_initial_pose_module.xacro (robot description, xacro)
@@ -41,14 +41,7 @@
       <parent link="${parent}"/>
       <child link="${prefix}_thigh"/>
-      <origin xyz="${x} ${y} ${z}" rpy="0 0 0"/>
+      <origin rpy="0 ${initial_hip_angle} 0" xyz="${x} ${y} ${z}"/>
       <axis xyz="0 1 0"/>
       <limit lower="-3.0" upper="1.0" effort="30.0" velocity="10.0"/>
-      <!-- 设置初始位置 -->
-      <xacro:if value="${mirror}">
-        <origin rpy="0 ${initial_hip_angle} 0" xyz="${x} ${y} ${z}"/>
-      </xacro:if>
-      <xacro:unless value="${mirror}">
-        <origin rpy="0 ${initial_hip_angle} 0" xyz="${x} ${y} ${z}"/>
-      </xacro:unless>
     </joint>
     <!-- ========== 小腿 (Shank) ========== -->
@@ -81,5 +74,5 @@
       <origin rpy="0 ${initial_knee_angle} 0" xyz="0 0 ${-thigh_length}"/>
       <axis xyz="0 1 0"/>
-      <limit lower="0.0" upper="3.0" effort="25.0" velocity="10.0"/>
+      <limit lower="0.0" upper="3.0" effort="50.0" velocity="10.0"/>
     </joint>
     <!-- ========== 轮子 (Wheel) ========== -->
